File: PCB/Wheelchair Powermeter PCB/Wheelchair Powermeter PCB.kicad_sch (KiCad schematic)
At the start: 25 parts, among them J1 USB4085-GF-A_REVB, U1 ESP32-V2, U2 TE4525, U3 4554_IMU_9DOF, U4 MPL3115A2

Commit message: Moooorrrrrrr
Parts:
- removed C1: C, Capacitor_THT:CP_Axial_L10.0mm_D4.5mm_P15.00mm_Horizontal, symbol Device:C
- removed TP3, TP4, TP5, TP6, TP7, TP8, TP_GND1, TP_GND2: TestPoint, TestPoint:TestPoint_Loop_D3.80mm_Drill2.5mm, symbol Connector:TestPoint
- removed U1: ESP32-V2, Adafruit:ESP32 V3, symbol Adafruit:ESP32-V2
- added U1: ESP32-S3, Adafruit:ESP32-S3, symbol Adafruit:ESP32-S3
- added U5: ~, Adafruit:SPI_Screen, symbol Adafruit:SPI_Screen
- R5, R6: value 100KR -> 100R
Connections:
- net 3.3V: now also U1.2 (3.3V), U1.3 (3.3V), U5.1 (3.3V)
- net GND: now also U1.4 (GND), U5.2 (GND)
- net SCL_MCU: now also U1.27 (SCL)
- net SDA_MCU: now also U1.28 (SDA)
- net POWER: now reaches J1.A4 (VBUS), J1.A9 (VBUS), J1.B4 (VBUS), J1.B9 (VBUS), TP_VBUS1.1
- net POWER: now also U1.17 (VBAT)
- net at S1.3 (NO_1), S1.4 (NO_2): now also U1.25 (D6)
- net at S2.3 (NO_1), S2.4 (NO_2): now also U1.26 (D5)
- new net: U1.11 (SCK), U5.3 (CK)
- new net: U1.12 (MOSI), U5.4 (SI)
- new net: U1.23 (D10), U5.5 (CS)
- new net: U1.22 (D11), U5.6 (RT)
- new net: U1.21 (D12), U5.7 (DC)
- new net: U1.20 (D13), U5.8 (BL)
Other:
- moved on the sheet: S1, S2, TP_3.3V1, TP_GND3, U2, U3A, U4
